File: Hardware/Proiect TSC v103.brd (EAGLE design)
At the start: 170.2 x 111.2 mm, 103 parts, among them IC1 BD5229G-TR, IC4 XC6220A331MR-G, J1 FH34SRJ-24S-0.5SH_99_, J2 SAMACSYS_PARTS_USB4110-GF-A, J3 QWIIC_RIGHT_ANGLE, J4 112A-TAAR-R03_ATTEND, Q1 20V/4.2A/52mΩ/1.4W, Q2 20V/4.2A/52mΩ/1.4W, Q3 SI1308EDL-T1-GE3, U1 W25Q512JVEIQ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

Commit message: Commit solving the issues
Routing:
- net SDA: track 208.6 -> 224.4 mm
- net FLASH_CS: track 88.1 -> 100.7 mm
- net 3V3: track 391.9 -> 403.9 mm
- net EPD_CS: track 125.0 -> 135.5 mm
- net EPD_3V3_C: track 111.2 -> 118.6 mm
- net EPD_BUSY: track 164.9 -> 169.8 mm
- net USB_D+: track 136.7 -> 140.1 mm
- net INT_RTC: track 146.6 -> 149.8 mm
- net EPD_3V3: track 66.1 -> 68.3 mm
- net SCK: track 198.6 -> 200.8 mm
- net EPD_RST: track 134.9 -> 136.5 mm
- net RX: track 47.0 -> 46.0 mm
- net GND: track 741.1 -> 741.0 mm, vias 20 -> 23
