File: Hardware/Proiect_TSC_v66.sch (EAGLE design)
At the start: 103 parts, among them IC1 BD5229G-TR, IC4 XC6220A331MR-G, J1 FH34SRJ-24S-0.5SH_99_, J2 SAMACSYS_PARTS_USB4110-GF-A, J3 QWIIC_RIGHT_ANGLE, J4 112A-TAAR-R03_ATTEND, Q1 20V/4.2A/52mΩ/1.4W, Q2 20V/4.2A/52mΩ/1.4W, Q3 SI1308EDL-T1-GE3, U1 W25Q512JVEIQ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

Commit message: Commit solving the issues
Other:
- moved on the sheet: BOOT_BUTTON, C1, C10, C10_SUPERCAP, C1_BAT, C1_BAT1, C1_BAT2, C2, C2_BAT, C3, C4, C4_USB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
